File: cyc1000_pidp-11_shim.kicad_pcb (KiCad board)
At the start: 4 copper layers, 95 x 61 mm, 88 parts, among them J1 FTDI_FRIEND, J11 Raspberry_Hat, J12 RS232_PMOD, J13 USD_PMOD, J14 ETH_PMOD, J4 EXTERNAL 5.0V POWER, U1 CYC1000

Commit message: Convert to KiCad 6
Other:
- net class Default removed
- net class Power removed
